File: iot_badge/iot_badge.sch (KiCad schematic (older format))
At the start: 18 parts

Commit message: work on power supplies and general schematics
Parts:
- removed BT?: Battery_Cell, symbol Device:Battery_Cell
- removed C? (x2): 4.7uF, symbol Device:CP
- removed D?: SDM02U30LP3-7B, symbol Device:D_Schottky
- removed J?: USB_C_Receptacle, symbol Connector:USB_C_Receptacle
- removed J?: Conn_01x02, symbol Connector_Generic:Conn_01x02
- removed PS?: XCL210C331GR-G, XCL219, symbol SamacSys_Parts:XCL210C331GR-G
- removed R?: 2k, symbol Device:R
- removed U?: MCP73831-2-OT, Package_TO_SOT_SMD:SOT-23-5, symbol Battery_Management:MCP73831-2-OT
- added C? (x2): C, Capacitor_SMD:C_0603_1608Metric, symbol pspice:C
- added C? (x2): 22pF, Capacitor_SMD:C_0603_1608Metric, symbol pspice:C
- added C? (x3): 10uF, Capacitor_SMD:C_0603_1608Metric, symbol pspice:C
- added D?: PMEG3005AESFYL, SamacSys_Parts:PMEG3005AESFYL, symbol Device:D_Schottky
- added FL?: ECMF02-4CMX8, ECMF024CMX8, symbol SamacSys_Parts:ECMF02-4CMX8
- added J?: USB_B_Micro, Connector_USB:USB_Micro-B_Molex-105133-0001, symbol Connector:USB_B_Micro
- added L?: 10uH, Inductor_SMD:L_0603_1608Metric, symbol Device:L
- added PS?: XCL210C331GR-G, XCL219, symbol SamacSys_Parts:XCL210C331GR-G
- added R?: 10k, Resistor_SMD:R_0603_1608Metric, symbol Device:R
- added U?: BAT-HLD-001, BATHLD001, symbol SamacSys_Parts:BAT-HLD-001
- added U?: MCP73831-2-OT, Package_TO_SOT_SMD:SOT-23-5, symbol Battery_Management:MCP73831-2-OT
- added Y?: FC-135 32.7680KA-A5, SamacSys_Parts:FC135327680KAA5, symbol Device:Crystal
- C? (x4): footprint (none) -> Capacitor_SMD:C_0603_1608Metric
- C?: value 10uF -> 22uF; footprint (none) -> Capacitor_SMD:C_0603_1608Metric
- D?: value SDM02U30LP3-7B -> PMEG3005AESFYL; footprint (none) -> SamacSys_Parts:PMEG3005AESFYL
- R? (x2): footprint (none) -> Resistor_SMD:R_0603_1608Metric
Connections:
- net labels added: +BATT, D+, D-, ID, L1, L2, NFC_L, SWDCLK, SWDIO, nCHARGE
- wire segments 0 -> 99
- no-connect marks 0 -> 4
Other:
- note added: "LIPO Charger"
- note added: "NRF52840"
- note added: "Power Supply"
- note added: "USB"
- moved on the sheet: C?, D?, IC?, R?

Commit message: add lipo holder, push-button and LEDs
Parts:
- removed C?: 10uF, Capacitor_SMD:C_0603_1608Metric, symbol pspice:C
- removed U?: BAT-HLD-001, BATHLD001, symbol SamacSys_Parts:BAT-HLD-001
- added C? (x5): 100nF, Capacitor_SMD:C_0603_1608Metric, symbol pspice:C
- added D? (x5): APA102-2020, LED_SMD:LED-APA102-2020, symbol LED:APA102-2020
- added J?: 1042P, 1042P, symbol SamacSys_Parts:1042P
- added R? (x5): 10k, Resistor_SMD:R_0603_1608Metric, symbol Device:R
- added S? (x5): EVQ-6Q202W, EVQ6Q202W, symbol SamacSys_Parts:EVQ-6Q202W
Connections:
- net labels added: -BATT, CKI_1, CKI_2, CKI_3, CKI_4, CKI_5, CKI_6, RESET, SDI_1, SDI_2, SDI_3, SDI_4, SDI_5, SDI_6, SW1, SW2, SW3, SW4
- wire segments 99 -> 185
- no-connect marks 4 -> 7
Other:
- note added: "Footprints from mouser library loader are sometimes shit..."
- note added: "LED APA102-2020"
- note added: "Push Button Switches"
- moved on the sheet: C?, D?, PS?, R?, U?

Commit message: connect motor driver and IMU
Parts:
- added C11: 10uF, Capacitor_SMD:C_0603_1608Metric, symbol pspice:C
- added C12, C17: 10nF, Capacitor_SMD:C_0603_1608Metric, symbol pspice:C
- added C13, C15, C18: 100nF, Capacitor_SMD:C_0603_1608Metric, symbol pspice:C
- added C16, C19: 2.2uF, Capacitor_SMD:C_0603_1608Metric, symbol pspice:C
- added J3, J4: Conn_01x02_Male, Connector_PinHeader_2.54mm:PinHeader_1x01_P2.54mm_Vertical, symbol Connector:Conn_01x02_Male
- added Q1: PMDPB30XN,115, SamacSys_Parts:PMDPB30XN115, symbol SamacSys_Parts:PMDPB30XN,115
- added R10: 2.2k, Resistor_SMD:R_0603_1608Metric, symbol Device:R
- added R11, R12: 0.5R, Resistor_SMD:R_0603_1608Metric, symbol Device:R
- added R8: 330R, Resistor_SMD:R_0603_1608Metric, symbol Device:R
- added U2: ICM-20602, Package_LGA:LGA-16_3x3mm_P0.5mm_LayoutBorder3x5y, symbol Sensor_Motion:ICM-20602
- added U3: BQ29700DSET, digikey-footprints:WFDFN-6_1.5x1.5mm, symbol dk_PMIC-Battery-Management:BQ29700DSET
- added U4: DRV8833PWPR, digikey-footprints:TSSOP-16-1EP_W4.40mm, symbol dk_PMIC-Full-Half-Bridge-Drivers:DRV8833PWPR
- FL1: renamed from FL?; footprint ECMF024CMX8 -> SamacSys_Parts:ECMF024CMX8
- IC1: renamed from IC?; footprint 113990582 -> SamacSys_Parts:113990582
- J2: renamed from J?; footprint 1042P -> SamacSys_Parts:1042P
- PS1: renamed from PS?; footprint XCL219 -> SamacSys_Parts:XCL219
- R9: renamed from R?; value 10k -> 2k
- S1, S2, S3, S4, S5: renamed from S?; footprint EVQ6Q202W -> SamacSys_Parts:EVQ6Q202W
- gave numbers to parts that had none: 34
Connections:
- net labels added: AIN_1, AIN_2, BIN_1, BIN_2, IMU_FSYNC, IMU_INT, IMU_MISO, IMU_MOSI, IMU_SCL, IMU_nCS, MA_1, MA_2, MB_1, MB_2, nFAULT, nSLEEP
- wire segments 185 -> 272
Other:
- note added: "1x18650 Battery Holder"
- note added: "Dual Motor Driver"
- note added: "IMU"
- moved on the sheet: C14, C20, C21, C22, C23, C24, D3, D4, D5, D6, D7, J2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

Commit message: add 5V boost supply for APA102 change some symbols to have nicer schematics
Parts:
- added C20: 10nF, Capacitor_SMD:C_0603_1608Metric, symbol pspice:C
- added C21, C22: 10uF, Capacitor_SMD:C_0603_1608Metric, symbol pspice:C
- added IC2: XCL103D503CR-G, XCL103D503CRG, symbol SamacSys_Parts:XCL103D503CR-G
- added R10, R14: 100k, Resistor_SMD:R_0603_1608Metric, symbol Device:R
- J3, J4: footprint Connector_PinHeader_2.54mm:PinHeader_1x01_P2.54mm_Vertical -> Connector_PinHeader_2.54mm:PinHeader_1x02_P2.54mm_Vertical
- renumbered C9 to C10, C20 to C23, C21 to C24, C22 to C25, C23 to C26, C24 to C27, C10 to C7, C7 to C8, C8 to C9, R10 to R11, R11 to R12, R12 to R13
Connections:
- net labels added: +5VL, V_BAT, V_BAT_ENA
- net labels removed: L1, L2
- wire segments 272 -> 311
Other:
- note added: "Battery measurement can\nbe enabled by uP by\nsetting GPIO to output low"
- note added: "LED Power Supply"
- note removed: "Footprints from mouser library loader are sometimes shit..."
- moved on the sheet: C10, C7, D1, D2, Q1

Commit message: refactor raytac NRF52840 symbol
Parts:
- removed C7: 22uF, Capacitor_SMD:C_0603_1608Metric, symbol pspice:C
- removed IC1: MDBT50Q-1MV2, SamacSys_Parts:113990582, symbol SamacSys_Parts:113990582
- removed L1: 10uH, Inductor_SMD:L_0603_1608Metric, symbol Device:L
- added C10, C11: 10uF, Capacitor_SMD:C_0603_1608Metric, symbol pspice:C
- added C12, C23, C24: 100nF, Capacitor_SMD:C_0603_1608Metric, symbol pspice:C
- added D3: LED, symbol Device:LED
- added IC1: MDBT50Q-1MV2, 113990582, symbol SamacSys_Parts:MDBT50Q-1MV2
- added R4: 1k, Resistor_SMD:R_0603_1608Metric, symbol Device:R
- added U3: SN74LVC2T45DCUR, Package_SO:VSSOP-8_2.4x2.1mm_P0.5mm, symbol Logic_LevelTranslator:SN74LVC2T45DCUR
- C5, C6: value 22pF -> 12pF
- R13: renamed from R14; value 100k -> 500k
- R6: renamed from R10; value 100k -> 500k
- renumbered C2 to C1, C20 to C15, C11 to C16, C12 to C17, C23 to C18, C24 to C19, C3 to C2, C25 to C20, C26 to C21, C27 to C22, C21 to C25, C15 to C26, C22 to C27, C16 to C28, C17 to C29, C4 to C3, C18 to C30, C19 to C31, C1 to C4, C8 to C7, C9 to C8, C10 to C9, D3 to D4, D4 to D5, D5 to D6, D6 to D7, D7 to D8, R5 to R10, R6 to R11, R7 to R12, R12 to R14, R13 to R15, R8 to R3, R9 to R5, R11 to R7, R3 to R8, R4 to R9, U3 to U2, U2 to U4, U4 to U5
Connections:
- net labels added: AREF, LED_CK, LED_SD, nRESET
- net labels removed: RESET, V_BAT_ENA
- wire segments 311 -> 347
- no-connect marks 7 -> 4
Other:
- note added: "3.7uA just for battery voltage\nmeasurement... Should put a P-MOS here\nN-MOS or GPO won't work as V_BAT would\ngo >VCC"
- note removed: "Battery measurement can\nbe enabled by uP by\nsetting GPIO to output low"
- moved on the sheet: C1, C14, C16, C17, C18, C19, C2, C20, C21, C22, C25, C26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
